File: PCB_Sim/PCB_Sim.kicad_pcb (KiCad board)
At the start: 2 copper layers, 95 x 72 mm, 12 parts, among them J1 Maneuver_ICS, J2 Loadcell_front_1, J3 Loadcell_front_2, J4 Loadcell_back_1, J5 Loadcell_back_2, J6 Speaker, SW1 SW_DPST_x2, U1 Pico

Commit message: Create PCB_HX711
HX711用取り付け基盤
Routing:
- net Net-(PAM1-in+): track 60.5 -> 51.9 mm
Changed lines of the file:
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@@
 	)
 	(segment
-		(start 171.45 91.44)
+		(start 172.72 92.71)
 		(end 173.99 93.98)
 		(width 0.2)
@@
 		(net 21)
 	)
-	(segment
-		(start 167.64 91.44)
-		(end 171.45 91.44)
-		(width 0.2)
-		(layer "F.Cu")
-		(net 21)
-	)
 	(via
-		(at 167.64 91.44)
+		(at 172.72 92.71)
 		(size 0.6)
 		(drill 0.3)
@@
 	)
 	(segment
+		(start 160.02 71.12)
+		(end 158.75 69.85)
+		(width 0.2)
+		(layer "B.Cu")
+		(net 21)
+	)
+	(segment
+		(start 171.45 91.44)
+		(end 163.83 91.44)
+		(width 0.2)
+		(layer "B.Cu")
+		(net 21)
+	)
+	(segment
+		(start 139.7 68.58)
+		(end 139.7 66.04)
+		(width 0.2)
+		(layer "B.Cu")
+		(net 21)
+	)
+	(segment
+		(start 163.83 91.44)
+		(end 160.02 87.63)
+		(width 0.2)
+		(layer "B.Cu")
+		(net 21)
+	)
+	(segment
 		(start 158.75 69.85)
 		(end 140.97 69.85)
@@
 	)
 	(segment
-		(start 163.83 91.44)
-		(end 160.02 87.63)
+		(start 172.72 92.71)
+		(end 171.45 91.44)
+		(width 0.2)
+		(layer "B.Cu")
+		(net 21)
+	)
+	(segment
+		(start 160.02 87.63)
+		(end 160.02 71.12)
 		(width 0.2)
 		(layer "B.Cu")
@@
 		(start 140.97 69.85)
 		(end 139.7 68.58)
-		(width 0.2)
-		(layer "B.Cu")
-		(net 21)
-	)
-	(segment
-		(start 160.02 71.12)
-		(end 158.75 69.85)
-		(width 0.2)
-		(layer "B.Cu")
-		(net 21)
-	)
-	(segment
-		(start 160.02 87.63)
-		(end 160.02 71.12)
-		(width 0.2)
-		(layer "B.Cu")
-		(net 21)
-	)
-	(segment
-		(start 139.7 68.58)
-		(end 139.7 66.04)
-		(width 0.2)
-		(layer "B.Cu")
-		(net 21)
-	)
-	(segment
-		(start 167.64 91.44)
-		(end 163.83 91.44)
 		(width 0.2)
 		(layer "B.Cu")
@@
 	)
 	(segment
+		(start 172.72 100.33)
+		(end 173.99 99.06)
+		(width 0.2)
+		(layer "F.Cu")
+		(net 73)
+	)
+	(segment
 		(start 173.99 99.06)
 		(end 177.8 99.06)
@@
 		(net 73)
 	)
-	(segment
-		(start 172.72 100.33)
-		(end 173.99 99.06)
-		(width 0.2)
-		(layer "F.Cu")
-		(net 73)
-	)
-	(segment
-		(start 172.72 105.41)
-		(end 172.72 100.33)
-		(width 0.2)
-		(layer "F.Cu")
-		(net 73)
-	)
-	(segment
-		(start 171.45 106.68)
-		(end 172.72 105.41)
-		(width 0.2)
-		(layer "F.Cu")
-		(net 73)
-	)
-	(segment
-		(start 162.56 106.68)
-		(end 171.45 106.68)
-		(width 0.2)
-		(layer "F.Cu")
-		(net 73)
-	)
 	(via
-		(at 162.56 106.68)
+		(at 172.72 100.33)
 		(size 0.6)
 		(drill 0.3)
@@
 	)
 	(segment
-		(start 148.59 105.41)
-		(end 148.59 102.87)
+		(start 171.45 101.6)
+		(end 127 101.6)
 		(width 0.2)
 		(layer "B.Cu")
@@
 	)
 	(segment
-		(start 162.56 106.68)
-		(end 149.86 106.68)
-		(width 0.2)
-		(layer "B.Cu")
-		(net 73)
-	)
-	(segment
-		(start 147.32 101.6)
-		(end 127 101.6)
-		(width 0.2)
-		(layer "B.Cu")
-		(net 73)
-	)
-	(segment
-		(start 149.86 106.68)
-		(end 148.59 105.41)
-		(width 0.2)
-		(layer "B.Cu")
-		(net 73)
-	)
-	(segment
-		(start 148.59 102.87)
-		(end 147.32 101.6)
-		(width 0.2)
-		(layer "B.Cu")
+		(start 172.72 100.33)
+		(end 171.45 101.6)
+		(width 0.2)
+		(layer "B.Cu")
