File: PCB_Sim/PCB_Sim.kicad_sch (KiCad schematic)
At the start: 7 parts, among them J1 Conn_01x04_Socket, J2 Conn_01x04_Socket, J3 Conn_01x04_Socket, J4 Conn_01x04_Socket, J5 Conn_01x03_Socket, J6 Conn_01x03_Socket, U1 Pico

Commit message: first commit with browser
ブラウザからのコミット
Parts:
- removed J5, J6: Conn_01x03_Socket, symbol Connector:Conn_01x03_Socket
- added D1: LED, 20241231Library:Padx2, symbol led:LED
- added J1: Maneuver_ICS, Footprints:JST_XH_S4B-XH-A_1x04_P2.50mm_Horizontal, symbol Connector:Conn_01x04_Socket
- added J6: Speaker, Footprints:JST_XH_S2B-XH-A_1x02_P2.50mm_Horizontal, symbol Connector:Conn_01x02_Socket
- added PAM1: PAM8012, Footprints:PAM8012, symbol pam8012:PAM8012
- added RV1: R_Potentiometer, 20241231Library:Padx3, symbol Device:R_Potentiometer
- added SW1: SW_DPST_x2, 20241231Library:Padx2, symbol Switch:SW_DPST_x2
- J2: renamed from J1; value Conn_01x04_Socket -> Loadcell_front_1; footprint (none) -> Footprints:JST_XH_S4B-XH-A_1x04_P2.50mm_Horizontal
- J3: renamed from J2; value Conn_01x04_Socket -> Loadcell_front_2; footprint (none) -> Footprints:JST_XH_S4B-XH-A_1x04_P2.50mm_Horizontal
- J4: renamed from J3; value Conn_01x04_Socket -> Loadcell_back_1; footprint (none) -> Footprints:JST_XH_S4B-XH-A_1x04_P2.50mm_Horizontal
- J5: renamed from J4; value Conn_01x04_Socket -> Loadcell_back_2; footprint (none) -> Footprints:JST_XH_S4B-XH-A_1x04_P2.50mm_Horizontal
- U1: footprint RPi_Pico:RPi_Pico_SMD_TH -> Footprints:RPi_Pico_SMD_TH
Connections:
- net DAT1: now reaches J2.3 (Pin_3)
- net DAT1: now also U1.5 (GPIO3)
- net 5V: now reaches J2.4 (Pin_4)
- net 5V: now also J3.4 (Pin_4), J4.4 (Pin_4), J5.4 (Pin_4), U1.40 (VBUS), J1.2 (Pin_2), PAM1.1 (+V)
- net DAT3: now reaches J4.3 (Pin_3)
- net DAT3: now also U1.10 (GPIO7)
- net DAT4: now reaches J5.3 (Pin_3)
- net DAT4: now also U1.12 (GPIO9)
- net CLK4: now reaches U1.11 (GPIO8)
- net CLK4: now also J5.2 (Pin_2)
- net O_SPK: now reaches U1.27 (GPIO21)
- net O_SPK: now also RV1.1
- net READY_LED: now reaches U1.29 (GPIO22)
- net READY_LED: now also D1.2 (A)
- net RESET_SW: now reaches U1.30 (RUN)
- net RESET_SW: now also SW1.2 (B)
- net GND: now reaches U1.38 (GND)
- net GND: now also J2.1 (Pin_1), J3.1 (Pin_1), J4.1 (Pin_1), J5.1 (Pin_1), D1.1 (K), J1.1 (Pin_1), PAM1.2 (GND), PAM1.4 (in-), RV1.3, SW1.1 (A)
- net DAT2: now reaches J3.3 (Pin_3)
- net DAT2: now also U1.7 (GPIO5)
- net DOUT1 renamed PRMT
- net PRMT: now also J1.4 (Pin_4); no longer J2.1 (Pin_1)
- removed net DOUT2: J3.1 (Pin_1), U1.5 (GPIO3)
- removed net DOUT3: J4.1 (Pin_1), U1.7 (GPIO5)
- removed net DOUT4: J5.1 (Pin_1), U1.10 (GPIO7)
- net SLK1 renamed CLK1
- net CLK1: now also U1.4 (GPIO2); no longer U1.1 (GPIO0)
- net SLK2 renamed CLK2
- net CLK2: now also U1.6 (GPIO4); no longer U1.4 (GPIO2)
- net SLK3 renamed CLK3
- net CLK3: now also U1.9 (GPIO6); no longer U1.6 (GPIO4)
- removed net SLK4: J5.2 (Pin_2), U1.9 (GPIO6)
- new net: PAM1.3 (in+), RV1.2
- new net PTMR: J1.3 (Pin_3), U1.1 (GPIO0)
- new net SPK+: J6.2 (Pin_2), PAM1.5 (SPK+)
- new net SPK-: J6.1 (Pin_1), PAM1.6 (SPK-)
- no-connect marks 0 -> 28
Other:
- moved on the sheet: J2, J3, J4, J5

Commit message: ver.2
Connections:
- net PRMT: now also U1.17 (GPIO13); no longer U1.2 (GPIO1)
- net PTMR: now also U1.16 (GPIO12); no longer U1.1 (GPIO0)
Changed lines of the file:
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@@
 	)
 	(no_connect
-		(at 132.08 105.41)
+		(at 132.08 67.31)
 	)
 	(no_connect
@@
 	)
 	(no_connect
-		(at 132.08 102.87)
+		(at 132.08 64.77)
 	)
 	(no_connect
@@
 	(wire
 		(pts
-			(xy 127 64.77) (xy 132.08 64.77)
+			(xy 127 102.87) (xy 132.08 102.87)
 		)
 		(stroke
@@
 	(wire
 		(pts
-			(xy 127 67.31) (xy 132.08 67.31)
+			(xy 127 105.41) (xy 132.08 105.41)
 		)
 		(stroke
@@
 	)
 	(label "PRMT"
-		(at 127 67.31 0)
+		(at 127 105.41 0)
 		(fields_autoplaced yes)
 		(effects
@@
 	)
 	(label "PTMR"
-		(at 127 64.77 0)
-		(fields_autoplaced yes)
-		(effects
+		(at 127 102.87 0)
+		(fields_autoplaced yes)
+		(effects
